File: 4bmc.sch (KiCad schematic (older format))
At the start: 136 parts

Commit message: major components are now connected
Connections:
- net labels removed: Reset
- wire segments 549 -> 762
Other:
- note added: "Instruction"
- note added: "Operand 1"
- note added: "Operand 2"
- note removed: "Register"
- moved on the sheet: U?, U?A, U?B, U?C, U?D

Commit message: added in/out labels, fixed J-K FF
Parts:
- removed U? (x3): 74LS04, symbol 74LS04
Connections:
- wire segments 762 -> 600
Other:
- note added: "Counter OUT"
- note added: "Data IN"
- note added: "Data OUT"
- note added: "Data Valid +"
